Commit message: feat(design): 几何基元扩展 + 22 关节编号图等 4 张工程图
外观（几何基元）
- 新增 design/geometry.py：6 种基元（box/rounded_box/cylinder/
  sphere/capsule/sphere_shell）+ 惯量解析式 + 三维变换（罗德里格斯）
  + 正交投影 + AABB 干涉检测，全部纯标准库
- robot_model.json 升级 v1.1：23 个 link 从清一色长方体改为
  球壳关节 + 胶囊连杆 + 圆角壳体 + 足底板，并补 label/group 字段
  包围盒与质量保持不变，故尺寸与仿真结果无回归

URDF
- visual 用真实基元，collision 用等效包围盒（标准工程做法）
- capsule→cylinder（长度含球头）、sphere_shell→sphere、rounded_box→box
- 惯量按基元形状解析计算，不再一律按长方体
- gen_urdf.py 新增几何合法性与"几何实测包络 vs 声明包络"校验

工程图（design/gen_drawings.py，纯标准库 SVG）
- 01_关节编号图 ★ 正视+侧视，22 关节全部编号，躯干 2 DOF 橙色高亮，
  附自由度构成、尺寸合规核验、22 关节明细表
- 02_三视图 正视/侧视/俯视 + 尺寸标注与官方上限对比
- 04_尺寸链图 头部链/左腿链逐级累加，总高校核 + 放置校核
- 05_舵机布局图 22 路舵机安装位置 + 按扭矩分档图例 + 汇总
- 图框、标题栏、尺寸线、单位与阶段标注齐全

一致性修复
- 舵机分档图例原先硬编码 6/4/12 路，与汇总表的 4/8/10 矛盾，
  现改为全部由模型数据推导，并加断言
- 关节明细表右边界原先与标题栏重叠，现收窄为 3 列并加回归测试

已验证
- 全量 133 项测试通过（原 87 + 新 46）
- 几何实测包络 475×190×110 mm 与声明值完全一致，足底 z=0
- 4 张图经 qlmanage 渲染后逐张目视核对，无越界/重叠
- 删净产出后从零复现全链路（URDF→图→仿真→扫描）

诚实性
- 图注明确标注：投影示意图，非 CAD 出图、非渲染图，尺寸为设计值
- 舵机参数标注 provisional，未建模效应单列

File: design/atri.urdf (robot description, URDF)
Before this commit: robot ATRI, 23 links, 22 joints
Links:
- link head_yaw_link: geometry collision box size=0.030000 0.030000 0.030000; visual cylinder length=0.030000 radius=0.015000
- link left_forearm: geometry collision box size=0.035000 0.035000 0.050000; visual cylinder length=0.050000 radius=0.017500
- link left_hip_roll_link: geometry collision box size=0.040000 0.040000 0.040000; visual sphere radius=0.020000
- link left_hip_yaw_link: geometry collision box size=0.040000 0.040000 0.040000; visual sphere radius=0.020000
- link left_shank: geometry collision box size=0.040000 0.040000 0.080000; visual cylinder length=0.080000 radius=0.020000
- link left_shoulder_pitch_link: geometry collision box size=0.040000 0.040000 0.040000; visual sphere radius=0.020000
- link left_thigh: geometry collision box size=0.045000 0.045000 0.080000; visual cylinder length=0.080000 radius=0.022500
- link left_upper_arm: geometry collision box size=0.040000 0.040000 0.060000; visual cylinder length=0.060000 radius=0.020000
- link right_forearm: geometry collision box size=0.035000 0.035000 0.050000; visual cylinder length=0.050000 radius=0.017500
- link right_hip_roll_link: geometry collision box size=0.040000 0.040000 0.040000; visual sphere radius=0.020000
- link right_hip_yaw_link: geometry collision box size=0.040000 0.040000 0.040000; visual sphere radius=0.020000
- link right_shank: geometry collision box size=0.040000 0.040000 0.080000; visual cylinder length=0.080000 radius=0.020000
- link right_shoulder_pitch_link: geometry collision box size=0.040000 0.040000 0.040000; visual sphere radius=0.020000
- link right_thigh: geometry collision box size=0.045000 0.045000 0.080000; visual cylinder length=0.080000 radius=0.022500
- link right_upper_arm: geometry collision box size=0.040000 0.040000 0.060000; visual cylinder length=0.060000 radius=0.020000
- link trunk_roll_link: geometry collision box size=0.035000 0.035000 0.030000; visual cylinder length=0.030000 radius=0.017500

Commit message: feat(design): 等轴测软件渲染器 + 连杆实体衔接修复
新增 design/gen_render.py（纯标准库软件渲染）
- 自研渲染管线：三角网格 -> 轴测投影 -> 画家算法深度排序
  -> 背面剔除 -> 平面着色（环境光 + 漫反射 + 边缘光）
- 无需 GPU / Blender / CAD，0.3 秒出 5 张图
- 输出 5 个视角：等轴测 / 正视 / 侧视 / 部位配色 / 背面
- 自然站姿（微屈膝、手臂外展）、地面网格、自动取景
- 附带 PNG 导出（macOS qlmanage，自动补正方形避免裁切）

geometry.py 新增
- mesh_box / mesh_cylinder / mesh_sphere / mesh_capsule / mesh()
- 全部网格已做水密性校验（每条边恰好被两个三角形共享）
- 修复圆柱端盖圆心错误（原先取了边缘点，导致端盖破面）

重大设计修复：连杆实体悬空
- 原先所有 link 几何都居中在关节坐标上，导致外形不连续：
  颈部有 55mm 空隙、踝部 27.5mm、腕部 17.5mm，
  渲染出来像"零件飘在空中"
- 新增 origin_mm（几何相对关节坐标系的偏移，等价 URDF visual origin）
- 逐个重算 23 个 link 的实体长度与偏移，使其从本关节延伸到下一关节
- 现在竖直链条零间隙，有回归测试 test_segments_connect_without_gaps
- URDF 的 visual/collision/inertial 均写出该偏移；
  非 Z 轴回转体自动补 rpy 摆正

外观调整
- 统一配色：白色外壳 + 深蓝灰关节壳 + 深色足底与夹爪
- 头部比例收敛（90x80 -> 76x68，高度不变，总高仍 475mm）

测试
- 新增网格水密性、渲染管线、相机约定等 15 项测试
- 全量 148 项通过（原 133 + 新 15）

诚实性
- 渲染图注明确标注：软件渲染设计示意图、非实机照片、尺寸为设计值

File: design/atri.urdf (robot description, URDF)
Before this commit: robot ATRI, 23 links, 22 joints
Links:
- link head_yaw_link: geometry collision box size=0.030000 0.030000 0.078000; visual cylinder length=0.078000 radius=0.015000
- link left_forearm: geometry collision box size=0.035000 0.035000 0.060000; visual cylinder length=0.060000 radius=0.017500
- link left_shank: geometry collision box size=0.040000 0.040000 0.087000; visual cylinder length=0.087000 radius=0.020000
- link left_thigh: geometry collision box size=0.045000 0.045000 0.090000; visual cylinder length=0.090000 radius=0.022500
- link left_upper_arm: geometry collision box size=0.040000 0.040000 0.070000; visual cylinder length=0.070000 radius=0.020000
- link right_forearm: geometry collision box size=0.035000 0.035000 0.060000; visual cylinder length=0.060000 radius=0.017500
- link right_shank: geometry collision box size=0.040000 0.040000 0.087000; visual cylinder length=0.087000 radius=0.020000
- link right_thigh: geometry collision box size=0.045000 0.045000 0.090000; visual cylinder length=0.090000 radius=0.022500
- link right_upper_arm: geometry collision box size=0.040000 0.040000 0.070000; visual cylinder length=0.070000 radius=0.020000

Commit message: feat(model): 新架构 v2 —— 身高对齐参考机 373 mm，质量改为真实分布
背景：v1 的 link 质量是"结构占位预算"（1650 g），不含 22 只舵机与电子件，
导出的 URDF 总质量 1.80 kg 而实物口径 2.26 kg —— 喂给刚体引擎的动力学是错的。

- gen_v2_baseline.py：v1→v2 一次性迁移，z ×0.785 → 身高 475→373 mm（对齐幻尔 TonyPi Pro）
- link 质量 = 结构 + 舵机 + 电子件 + 分摊线束；sum(link mass) = 2146 g，质量闭合 ±0 g
- URDF 新增 22 只舵机的 visual/collision 附加体（球关节壳包不住 45.2 mm 舵机，实物靠支架夹持）
- 新增 design/placements.json：22 舵机 + 10 电子件 + 23 结构件的宿主/坐标/尺寸/质量
- 新增 design/reference/tonypi_pro_baseline.json：参考机公开参数与可迁移结论
- 扭矩判据改用「堵转 × 50% = 1.47 N·m」（依据参考机 1.8 kg 用 1.67 N·m 堵转舵机可行走），
  弃用无权威出处的「额定 1.0 N·m」；腿关节需求 1.11→1.05 N·m，占新判据 71%
- 新增 gen_spec_sheet.py 渲染《新架构参数总表》（人看的视图，禁止手工维护）
- 修 CI 历史红：交接包附件 PNG→SVG 回退（PNG 被 gitignore，全新 clone 必红）；
  测试不再硬编码 475 mm 与舵机几何，改为从模型推导
- 订正 TonyPi 参考文档中未做尺寸折算的结构质量结论

File: design/atri.urdf (robot description, URDF)
Before this commit: robot ATRI, 23 links, 22 joints
Links:
- link head: mass 0.120000 -> 0.061820; geometry collision box size=0.076000 0.068000 0.043200; visual box size=0.076000 0.068000 0.043200
- link head_yaw_link: mass 0.030000 -> 0.073290; geometry collision box size=0.030000 0.030000 0.061200; collision box size=0.045200 0.024700 0.035000
- link left_foot: mass 0.085000 -> 0.032670; geometry collision box size=0.110000 0.060000 0.019600; visual box size=0.110000 0.060000 0.019600
- link left_forearm: mass 0.055000 -> 0.074860; geometry collision box size=0.035000 0.035000 0.054600; collision box size=0.045200 0.024700 0.035000
- link left_gripper: mass 0.030000 -> 0.010090; geometry collision box size=0.050000 0.030000 0.019600; visual box size=0.050000 0.030000 0.019600
- link left_hip_roll_link: mass 0.040000 -> 0.071910; geometry collision box size=0.037200 0.037200 0.037200; collision box size=0.045200 0.024700 0.035000
- link left_hip_yaw_link: mass 0.040000 -> 0.071910; geometry collision box size=0.037200 0.037200 0.037200; collision box size=0.045200 0.024700 0.035000
- link left_shank: mass 0.070000 -> 0.083750; geometry collision box size=0.040000 0.040000 0.076900; collision box size=0.045200 0.024700 0.035000
- link left_shoulder_pitch_link: mass 0.040000 -> 0.071910; geometry collision box size=0.037200 0.037200 0.037200; collision box size=0.045200 0.024700 0.035000
- link left_thigh: mass 0.080000 -> 0.088690; geometry collision box size=0.045000 0.045000 0.080300; collision box size=0.045200 0.024700 0.035000
- link left_upper_arm: mass 0.075000 -> 0.080250; geometry collision box size=0.040000 0.040000 0.063600; collision box size=0.045200 0.024700 0.035000
- link pelvis: mass 0.130000 -> 0.225160; geometry collision box size=0.045200 0.024700 0.035000; collision box size=0.045200 0.024700 0.035000
- link right_foot: mass 0.085000 -> 0.032670; geometry collision box size=0.110000 0.060000 0.019600; visual box size=0.110000 0.060000 0.019600
- link right_forearm: mass 0.055000 -> 0.074860; geometry collision box size=0.035000 0.035000 0.054600; collision box size=0.045200 0.024700 0.035000
- link right_gripper: mass 0.030000 -> 0.010090; geometry collision box size=0.050000 0.030000 0.019600; visual box size=0.050000 0.030000 0.019600
- link right_hip_roll_link: mass 0.040000 -> 0.071910; geometry collision box size=0.037200 0.037200 0.037200; collision box size=0.045200 0.024700 0.035000
- link right_hip_yaw_link: mass 0.040000 -> 0.071910; geometry collision box size=0.037200 0.037200 0.037200; collision box size=0.045200 0.024700 0.035000
- link right_shank: mass 0.070000 -> 0.083750; geometry collision box size=0.040000 0.040000 0.076900; collision box size=0.045200 0.024700 0.035000
- link right_shoulder_pitch_link: mass 0.040000 -> 0.071910; geometry collision box size=0.037200 0.037200 0.037200; collision box size=0.045200 0.024700 0.035000
- link right_thigh: mass 0.080000 -> 0.088690; geometry collision box size=0.045000 0.045000 0.080300; collision box size=0.045200 0.024700 0.035000
- link right_upper_arm: mass 0.075000 -> 0.080250; geometry collision box size=0.040000 0.040000 0.063600; collision box size=0.045200 0.024700 0.035000
- link torso_upper: mass 0.300000 -> 0.545920; geometry collision box size=0.045200 0.024700 0.035000; collision box size=0.045200 0.024700 0.035000
- link trunk_roll_link: mass 0.040000 -> 0.067720; geometry collision box size=0.035000 0.035000 0.023600; collision box size=0.045200 0.024700 0.035000
Joints:
- joint head_pitch: origin xyz=0.000000 0.000000 0.035000 rpy=0 0 0 -> xyz=0.000000 0.000000 0.027500 rpy=0 0 0
- joint head_yaw: origin xyz=0.000000 0.000000 0.105000 rpy=0 0 0 -> xyz=0.000000 0.000000 0.082400 rpy=0 0 0
- joint left_ankle_pitch: origin xyz=0.000000 0.000000 -0.080000 rpy=0 0 0 -> xyz=0.000000 0.000000 -0.062800 rpy=0 0 0
- joint left_elbow_pitch: origin xyz=0.000000 0.000000 -0.060000 rpy=0 0 0 -> xyz=0.000000 0.000000 -0.047100 rpy=0 0 0
- joint left_gripper: origin xyz=0.000000 0.000000 -0.050000 rpy=0 0 0 -> xyz=0.000000 0.000000 -0.039200 rpy=0 0 0
- joint left_hip_pitch: origin xyz=0.000000 0.000000 -0.025000 rpy=0 0 0 -> xyz=0.000000 0.000000 -0.019600 rpy=0 0 0
- joint left_hip_roll: origin xyz=0.000000 0.000000 -0.025000 rpy=0 0 0 -> xyz=0.000000 0.000000 -0.019600 rpy=0 0 0
- joint left_hip_yaw: origin xyz=0.000000 0.045000 -0.025000 rpy=0 0 0 -> xyz=0.000000 0.045000 -0.019600 rpy=0 0 0
- joint left_knee_pitch: origin xyz=0.000000 0.000000 -0.080000 rpy=0 0 0 -> xyz=0.000000 0.000000 -0.062800 rpy=0 0 0
- joint left_shoulder_pitch: origin xyz=0.000000 0.075000 0.015000 rpy=0 0 0 -> xyz=0.000000 0.075000 0.011800 rpy=0 0 0
- joint right_ankle_pitch: origin xyz=0.000000 0.000000 -0.080000 rpy=0 0 0 -> xyz=0.000000 0.000000 -0.062800 rpy=0 0 0
- joint right_elbow_pitch: origin xyz=0.000000 0.000000 -0.060000 rpy=0 0 0 -> xyz=0.000000 0.000000 -0.047100 rpy=0 0 0
- joint right_gripper: origin xyz=0.000000 0.000000 -0.050000 rpy=0 0 0 -> xyz=0.000000 0.000000 -0.039200 rpy=0 0 0
- joint right_hip_pitch: origin xyz=0.000000 0.000000 -0.025000 rpy=0 0 0 -> xyz=0.000000 0.000000 -0.019600 rpy=0 0 0
- joint right_hip_roll: origin xyz=0.000000 0.000000 -0.025000 rpy=0 0 0 -> xyz=0.000000 0.000000 -0.019600 rpy=0 0 0
- joint right_hip_yaw: origin xyz=0.000000 -0.045000 -0.025000 rpy=0 0 0 -> xyz=0.000000 -0.045000 -0.019600 rpy=0 0 0
- joint right_knee_pitch: origin xyz=0.000000 0.000000 -0.080000 rpy=0 0 0 -> xyz=0.000000 0.000000 -0.062800 rpy=0 0 0
- joint right_shoulder_pitch: origin xyz=0.000000 -0.075000 0.015000 rpy=0 0 0 -> xyz=0.000000 -0.075000 0.011800 rpy=0 0 0
- joint trunk_pitch: origin xyz=0.000000 0.000000 0.035000 rpy=0 0 0 -> xyz=0.000000 0.000000 0.027500 rpy=0 0 0
- joint trunk_roll: origin xyz=0.000000 0.000000 0.025000 rpy=0 0 0 -> xyz=0.000000 0.000000 0.019600 rpy=0 0 0

Commit message: feat(model): v3 —— 数据口径切到协作者 CAD 实装测量
按用户决定：相关数据以协作者最新上传的 CAD 实装结果为准（提交 6d4b077 /
项目文档/骨架结构与集成方案.md §6–§7）。

L1 模型（v2 → v3，gen_v3_baseline.py）
- 结构件 500 → 1790 g（真实 CAD 体积 × PETG 1.27 g/cm³，74 个件）
- 整机 2146 → 3437 g；踝关节需求 1.037 → 1.629 N·m（占「堵转×50%」判据 111% ❌）
- 新增 installed_envelope_mm = 418 × 223 × 129 mm（CAD 实装；基元/运动学口径仍 372.8）
- 新增 reduction_paths：A 拓扑减重 900–1100 g / B 买金属件 550–700 g / C 减自由度
- 新增 design/reference/cad_assembly_measurements.json（机器可读的实装测量）
- 新增 design/gen_placements.py：placements.json 改为常规产物（原来内嵌在 v2 一次性迁移里，v3 改质量后就过期了）

同步上游 6d4b077 的实物订正
- 舵机空载速度 300 → 270 °/s（0.222 s/60°，来源实物包装标签 ST-3215-C018）
  同步到 robot_model.json / servo_spec.json / components.json / domain_random.json

文档与产出全量同步到 v3 口径（41.8 cm / 3437 g / 111% / 减重路径）
- 技术方案、项目综述、BOM与阶段性指标、材料上传准备、答辩Q&A
- 答辩PPT-逐页文案-v3（v3.2 修订说明）、答辩PPT-交付说明、答辩PPT-待回填清单
- 三个交接 Prompt、外观尺寸零件设计Prompt、设计数据包Prompt、TonyPi 参考文档
- 根 README、design/README、design/cad/README、design/cad/build_all.py 预算常量
- ppt/build_deck.py 重新出片（51 页，版面自检 0 问题）
- webots 世界重新生成、软件 config/robot.json 同步

说明：PDF 按用户决定暂不导出（材料仍会持续改动）。

File: design/atri.urdf (robot description, URDF)
Before this commit: robot ATRI, 23 links, 22 joints
Links:
- link head: mass 0.061820 -> 0.155100
- link head_yaw_link: mass 0.073290 -> 0.109600
- link left_foot: mass 0.032670 -> 0.114300
- link left_forearm: mass 0.074860 -> 0.115200
- link left_gripper: mass 0.010090 -> 0.035200
- link left_hip_roll_link: mass 0.071910 -> 0.104900
- link left_hip_yaw_link: mass 0.071910 -> 0.104900
- link left_shank: mass 0.083750 -> 0.146400
- link left_shoulder_pitch_link: mass 0.071910 -> 0.104900
- link left_thigh: mass 0.088690 -> 0.163400
- link left_upper_arm: mass 0.080250 -> 0.134200
- link pelvis: mass 0.225160 -> 0.339600
- link right_foot: mass 0.032670 -> 0.114300
- link right_forearm: mass 0.074860 -> 0.115200
- link right_gripper: mass 0.010090 -> 0.035200
- link right_hip_roll_link: mass 0.071910 -> 0.104900
- link right_hip_yaw_link: mass 0.071910 -> 0.104900
- link right_shank: mass 0.083750 -> 0.146400
- link right_shoulder_pitch_link: mass 0.071910 -> 0.104900
- link right_thigh: mass 0.088690 -> 0.163400
- link right_upper_arm: mass 0.080250 -> 0.134200
- link torso_upper: mass 0.545920 -> 0.695500
- link trunk_roll_link: mass 0.067720 -> 0.090000

Commit message: feat(model)!: 质量口径回灌到 CAD 实测（URDF/模型/世界 3.4366→3.0367 kg）
线程产物（主会话已复验）：
- 数据源 cad_assembly_measurements.json → 结构 1390.4 g/81 件、包络 160×268×407、整机 3036.4 g
- robot_model.json / atri.urdf / atri_22dof.wbt 三处拉齐；'整机重量方案未定案'标记全程保留
- 运动学零变化：22 关节 × 10 字段 220 项差异 0，关节段逐字节一致；
  URDF 改动仅 23 mass + 23 inertia，世界仅 23 mass 行（掩码后逐字节一致）

连带修正（主会话）：
- gen_spec_sheet.py / check_fit.py / robot.json 硬编码 1490/3136/1.90 全部跟随
- gen_v3_baseline.py history 增加'第 6–10 轮合入后'一节（注：_refresh 路径有意保留既有
  history 以免重复灌条目，故 robot_model.json 里当前条目名仍是'第 5 轮后（当前）'，为已知
  1 行文案瑕疵，留待重迁移时生效）
- test_handoff.py: '3.136'→'3.036'；续航断言改为**自洽判据**（consumed=I×h、
  required=consumed/0.8 + 量级区间），并保留'缺口必须写明'的约束
- test_design_package.py docstring 1490→1390

新口径（质量变小后联动）：平均电流 18.92→**18.42 A**、30 min 需求 11.83→**11.52 Ah**、
整包 1.19→**1.16 kg**；URDF sum=3.0367 kg。

⚠️ 力矩：踝 1.492→**1.446 N·m（147.5%）**、trunk_roll 1.899→**1.835 N·m（187.2%）**，
但线程查出 perpendicular_arm() 把竖直分量算进力臂 —— trunk_roll 高估 2.02×
（修正后 92.5%，会从'超额定'变'不超'），trunk_pitch 真值应为 0，已标'待复核'。

⚠️ 未提交（有意）：design/placements.json 重生成后有 74 处字段差异（IMU 移到骨盆、
相机罩轴向修正），会动到装配基准；为不干扰正在跑的足部线程，已回退，待其收口后
单独重生成 + 全量复验（❌=0 必须重新确认）。

测试：软件全量 432 项 OK；Webots 离线桩 40 项 OK。

File: design/atri.urdf (robot description, URDF)
Before this commit: robot ATRI, 23 links, 22 joints
Links:
- link head: mass 0.155100 -> 0.126400
- link head_yaw_link: mass 0.109600 -> 0.098400
- link left_foot: mass 0.114300 -> 0.089200
- link left_forearm: mass 0.115200 -> 0.102800
- link left_gripper: mass 0.035200 -> 0.027500
- link left_hip_roll_link: mass 0.104900 -> 0.094600
- link left_hip_yaw_link: mass 0.104900 -> 0.094600
- link left_shank: mass 0.146400 -> 0.127000
- link left_shoulder_pitch_link: mass 0.104900 -> 0.094600
- link left_thigh: mass 0.163400 -> 0.140300
- link left_upper_arm: mass 0.134200 -> 0.117500
- link pelvis: mass 0.339600 -> 0.304000
- link right_foot: mass 0.114300 -> 0.089200
- link right_forearm: mass 0.115200 -> 0.102800
- link right_gripper: mass 0.035200 -> 0.027500
- link right_hip_roll_link: mass 0.104900 -> 0.094600
- link right_hip_yaw_link: mass 0.104900 -> 0.094600
- link right_shank: mass 0.146400 -> 0.127000
- link right_shoulder_pitch_link: mass 0.104900 -> 0.094600
- link right_thigh: mass 0.163400 -> 0.140300
- link right_upper_arm: mass 0.134200 -> 0.117500
- link torso_upper: mass 0.695500 -> 0.648600
- link trunk_roll_link: mass 0.090000 -> 0.083100
