Commit message: 更新装配快照、URDF 与零件表，去掉第二块电池

File: design/v2/out/sim/atri_v2.urdf (robot description, URDF)
Before this commit: robot atri_v2, 21 links, 20 joints
Joints:
- joint left_gripper: origin xyz=0.000000 0.000000 -0.052000 rpy=0 0 0 -> xyz=0.000000 0.000000 -0.060000 rpy=0 0 0
- joint right_gripper: origin xyz=0.000000 0.000000 -0.052000 rpy=0 0 0 -> xyz=0.000000 0.000000 -0.060000 rpy=0 0 0

Commit message: 设计：连杆惯量按采购件与脚底板，不再摊成实心盒
20 只舵机、电池和 Pi 放图纸坐标；脚用 2 mm 铝板加 TPU 鞋底，
其余结构按非脚包围盒体积分配。不是称重，也不是 CAD 网格惯量。

File: design/v2/out/sim/atri_v2.urdf (robot description, URDF)
Before this commit: robot atri_v2, 21 links, 20 joints
Links:
- link head: mass 0.132336 -> 0.153286; geometry collision box size=0.0560 0.0560 0.0480; visual box size=0.0560 0.0560 0.0480
- link head_yaw_link: mass 0.039701 -> 0.072629; geometry collision box size=0.0300 0.0300 0.0300; visual box size=0.0300 0.0300 0.0300
- link left_foot: mass 0.105869 -> 0.120360; geometry collision box size=0.1200 0.0700 0.0440; visual box size=0.1200 0.0700 0.0440
- link left_fore: mass 0.066168 -> 0.069104; geometry collision box size=0.0180 0.0200 0.0600; visual box size=0.0180 0.0200 0.0600
- link left_grip: mass 0.031761 -> 0.060955; geometry collision box size=0.0120 0.0200 0.0380; visual box size=0.0120 0.0200 0.0380
- link left_hand: mass 0.039701 -> 0.069104; geometry collision box size=0.0180 0.0200 0.0600; visual box size=0.0180 0.0200 0.0600
- link left_hip_roll_link: mass 0.052934 -> 0.072629; geometry collision box size=0.0300 0.0300 0.0300; visual box size=0.0300 0.0300 0.0300
- link left_shank: mass 0.119102 -> 0.077409; geometry collision box size=0.0220 0.0200 0.0780; visual box size=0.0220 0.0200 0.0780
- link left_thigh: mass 0.145570 -> 0.077409; geometry collision box size=0.0220 0.0200 0.0780; visual box size=0.0220 0.0200 0.0780
- link left_upper: mass 0.079402 -> 0.073178; geometry collision box size=0.0200 0.0240 0.0580; visual box size=0.0200 0.0240 0.0580
- link pelvis: mass 0.211738 -> 0.098725; geometry collision box size=0.0900 0.0700 0.0240; visual box size=0.0900 0.0700 0.0240
- link right_foot: mass 0.105869 -> 0.120360; geometry collision box size=0.1200 0.0700 0.0440; visual box size=0.1200 0.0700 0.0440
- link right_fore: mass 0.066168 -> 0.069104; geometry collision box size=0.0180 0.0200 0.0600; visual box size=0.0180 0.0200 0.0600
- link right_grip: mass 0.031761 -> 0.060955; geometry collision box size=0.0120 0.0200 0.0380; visual box size=0.0120 0.0200 0.0380
- link right_hand: mass 0.039701 -> 0.069104; geometry collision box size=0.0180 0.0200 0.0600; visual box size=0.0180 0.0200 0.0600
- link right_hip_roll_link: mass 0.052934 -> 0.072629; geometry collision box size=0.0300 0.0300 0.0300; visual box size=0.0300 0.0300 0.0300
- link right_shank: mass 0.119102 -> 0.077409; geometry collision box size=0.0220 0.0200 0.0780; visual box size=0.0220 0.0200 0.0780
- link right_thigh: mass 0.145570 -> 0.077409; geometry collision box size=0.0220 0.0200 0.0780; visual box size=0.0220 0.0200 0.0780
- link right_upper: mass 0.079402 -> 0.073178; geometry collision box size=0.0200 0.0240 0.0580; visual box size=0.0200 0.0240 0.0580
- link torso: mass 0.582278 -> 0.683436; geometry collision box size=0.1000 0.0800 0.0780; visual box size=0.1000 0.0800 0.0780
- link trunk_roll_link: mass 0.052934 -> 0.072629; geometry collision box size=0.0300 0.0300 0.0300; visual box size=0.0300 0.0300 0.0300
